File: KiCAD/chipcon.sch (KiCad schematic (older format))
At the start: 37 parts, among them CON1 BARREL_JACK, J1 audio_out, J2 video out, P1 SD card, P2 ICSP, SW1 reset, SW2 power, U1 ATMEGA328-PU, U2 23LC512, U3 LT1117-3,3, X1 16Mhz, k1 KEYPAD

Commit message: travail sur schématique,ccasm,chip-dasm
Parts:
- R1: value 4k7 -> 10K
- renumbered C9 to C10, C10 to C11, C11 to C5, C5 to C6, C6 to C7, C7 to C8, C8 to C9, R9 to R10, R10 to R7, R7 to R8, R8 to R9
Changed lines of the file:
@@
 Sheet 1 1
 Title ""
-Date "24 oct 2014"
+Date "30 oct 2014"
 Rev ""
 Comp ""
@@
 $EndComp
 $Comp
-L C C5
+L C C6
 U 1 1 542046E9
 P 8300 6150
-F 0 "C5" H 8350 6250 50  0000 L CNN
+F 0 "C6" H 8350 6250 50  0000 L CNN
 F 1 "1µF" H 8350 6050 50  0000 L CNN
 F 2 "~" H 8300 6150 60  0000 C CNN
@@
 $EndComp
 $Comp
-L C C9
+L C C10
 U 1 1 54204742
 P 9850 6000
-F 0 "C9" H 9900 6100 50  0000 L CNN
+F 0 "C10" H 9900 6100 50  0000 L CNN
 F 1 "100nF" H 9900 5900 50  0000 L CNN
 F 2 "~" H 9850 6000 60  0000 C CNN
@@
 AVCC
 $Comp
-L C C10
+L C C11
 U 1 1 542048CE
 P 10300 6000
-F 0 "C10" H 10350 6100 50  0000 L CNN
+F 0 "C11" H 10350 6100 50  0000 L CNN
 F 1 "1µF" H 10350 5900 50  0000 L CNN
 F 2 "~" H 10300 6000 60  0000 C CNN
@@
 $EndComp
 $Comp
-L C C6
+L C C7
 U 1 1 542048DA
 P 8550 6150
-F 0 "C6" H 8600 6250 50  0000 L CNN
+F 0 "C7" H 8600 6250 50  0000 L CNN
 F 1 "100nF" H 8600 6050 50  0000 L CNN
 F 2 "~" H 8550 6150 60  0000 C CNN
@@
 $EndComp
 $Comp
-L R R7
+L R R8
 U 1 1 54204BAE
 P 8150 2750
-F 0 "R7" V 8230 2750 50  0000 C CNN
+F 0 "R8" V 8230 2750 50  0000 C CNN
 F 1 "10K" V 8150 2750 50  0000 C CNN
 F 2 "~" H 8150 2750 60  0000 C CNN
@@
 $EndComp
 $Comp
-L R R8
+L R R9
 U 1 1 54204BC8
 P 8350 2750
-F 0 "R8" V 8430 2750 50  0000 C CNN
+F 0 "R9" V 8430 2750 50  0000 C CNN
 F 1 "10K" V 8350 2750 50  0000 C CNN
 F 2 "~" H 8350 2750 60  0000 C CNN
@@
 3,3V
 $Comp
-L C C7
+L C C8
 U 1 1 54205F28
 P 9050 6150
-F 0 "C7" H 9100 6250 50  0000 L CNN
+F 0 "C8" H 9100 6250 50  0000 L CNN
 F 1 "100nF" H 9100 6050 50  0000 L CNN
 F 2 "~" H 9050 6150 60  0000 C CNN
@@
 P 2300 3950
 F 0 "R1" V 2380 3950 50  0000 C CNN
-F 1 "4k7" V 2300 3950 50  0000 C CNN
+F 1 "10K" V 2300 3950 50  0000 C CNN
 F 2 "~" H 2300 3950 60  0000 C CNN
 F 3 "~" H 2300 3950 60  0000 C CNN
@@
 3,3V
 $Comp
-L C C8
+L C C9
 U 1 1 543B1CFB
 P 9400 3100
-F 0 "C8" H 9450 3200 50  0000 L CNN
+F 0 "C9" H 9450 3200 50  0000 L CNN
 F 1 "100nF" H 9450 3000 50  0000 L CNN
 F 2 "~" H 9400 3100 60  0000 C CNN
@@
 	8550 2500 8150 2500
 $Comp
-L R R9
+L R R10
 U 1 1 5443FC07
 P 9450 5750
-F 0 "R9" V 9530 5750 50  0000 C CNN
+F 0 "R10" V 9530 5750 50  0000 C CNN
 F 1 "10R" V 9450 5750 50  0000 C CNN
 F 2 "~" H 9450 5750 60  0000 C CNN
@@
 	10300 6200 10300 6300
 $Comp
-L ELECTROLYTIC C11
+L ELECTROLYTIC C5
 U 1 1 5445B724
 P 7900 6350
-F 0 "C11" H 7750 6600 60  0000 C CNN
+F 0 "C5" H 7750 6600 60  0000 C CNN
 F 1 "10µF/16V" H 7650 6250 60  0000 C CNN
 F 2 "~" H 7900 6350 60  0000 C CNN
@@
 $EndComp
 $Comp
-L R R10
+L R R7
 U 1 1 5449B415
 P 7700 5500
-F 0 "R10" V 7780 5500 50  0000 C CNN
+F 0 "R7" V 7780 5500 50  0000 C CNN
 F 1 "100R" V 7700 5500 50  0000 C CNN
 F 2 "~" H 7700 5500 60  0000 C CNN
